Commit message: 新增前後萬向輪

File: my_diffcar/urdf/diffcar.xacro (robot description, xacro)
@@ -89,4 +89,40 @@
   <axis xyz="1 0 0" />
 </joint>
+<!-- front caster link -->
+<link name="front_caster_link">
+  <visual>
+    <geometry>
+      <sphere radius="${(wheel_radius - thickness/2)/2}" />
+    </geometry>
+    <origin xyz="0 0 0" rpy="0 0 0" />
+    <material name="black">
+      <color rgba="0 0 0 1"/>
+    </material>
+  </visual>
+</link>
+<joint name="joint_front_caster" type="continuous">
+<parent link="base_link" />
+<child link="front_caster_link" />
+<origin xyz="0 ${height/2} ${(wheel_radius - thickness/2)/2}" rpy="0 0 0" />
+<axis xyz="1 0 0" />
+</joint>
+<!-- back caster link -->
+<link name="back_caster_link">
+  <visual>
+    <geometry>
+      <sphere radius="${(wheel_radius - thickness/2)/2}" />
+    </geometry>
+    <origin xyz="0 0 0" rpy="0 0 0" />
+    <material name="black">
+      <color rgba="0 0 0 1"/>
+    </material>
+  </visual>
+</link>
+<joint name="joint_back_caster" type="continuous">
+<parent link="base_link" />
+<child link="back_caster_link" />
+<origin xyz="0 ${-height/2} ${(wheel_radius - thickness/2)/2}" rpy="0 0 0" />
+<axis xyz="1 0 0" />
+</joint>
 <transmission name="left_tran">
   <type>transmission_interface/SimpleTransmission</type>

Commit message: 將輪子用巨集表示

File: my_diffcar/urdf/diffcar.xacro (robot description, xacro)
@@ -4,4 +4,5 @@
 <xacro:property name="PI" value="3.1415926" />
 <xacro:property name="mass" value="1" /> <!-- kg -->
+<xacro:property name="wheel_mass" value="0.3" /> <!-- kg -->
 <xacro:property name="width" value="0.2" /> <!-- 0.1m -->
 <xacro:property name="height" value="0.4" /> <!-- 0.2m -->
@@ -9,5 +10,78 @@
 <xacro:property name="wheel_thickness" value="0.02" /> <!-- 1 cm -->
 <xacro:property name="wheel_radius" value="0.05" /> <!-- 5 cm -->
+<!-- define macros -->
+<xacro:macro name="sphere_inertial_matrix_" params="m r">
+  <inertial>
+    <mass value="${m}" />
+    <inertia ixx="${2*m*r*r/5}" ixy="0" ixz="0"
+             iyy="${2*m*r*r/5}" iyz="0"
+             izz="${2*m*r*r/5}" />
+    </inertial>
+</xacro:macro>
+<xacro:macro name="cylinder_inertial_matrix_" params="m r h">
+  <inertial>
+    <mass value="${m}" />
+    <inertia ixx="${m*(3*r*r+h*h)/12}" ixy = "0" ixz = "0"
+             iyy="${m*(3*r*r+h*h)/12}" iyz = "0"
+             izz="${m*r*r/2}" />
+  </inertial>
+</xacro:macro>
+<xacro:macro name="wheel_" params="prefix reflect">
+<link name="${prefix}_wheel_link">
+  <visual>
+    <geometry>
+      <cylinder length="${wheel_thickness}" radius="${wheel_radius}" />
+    </geometry>
+    <origin xyz="0 0 0" rpy="0 ${PI/2} 0" />
+    <material name="blue">
+      <color rgba="0 0 .8 1"/>
+    </material>
+  </visual>
+  <collision>
+    <geometry>
+      <cylinder length="${wheel_thickness}" radius="${wheel_radius}" />
+    </geometry>
+    <origin xyz="0 0 0" rpy="0 ${PI/2} 0" />
+  </collision>
+  <cylinder_inertial_matrix_  m="${wheel_mass}" r="${wheel_radius}" h="${wheel_thickness}" />
+</link>
+<gazebo reference="${prefix}_wheel_link">
+  <material>Gazebo/Blue</material>
+</gazebo>
+<joint name="${prefix}_wheel_joint" type="continuous">
+  <parent link="base_link" />
+  <child link="${prefix}_wheel_link" />
+  <origin xyz="${(width/2 + wheel_thickness/2)*reflect} 0 ${wheel_radius}" rpy="0 0 0" />
+  <axis xyz="1 0 0" />
+</joint>
+<transmission name="${prefix}_tran">
+  <type>transmission_interface/SimpleTransmission</type>
+  <joint name="${prefix}_whell_joint">
+    <hardwareInterface>hardware_interface/VelocityJointInterface</hardwareInterface>
+  </joint>
+  <actuator name="${prefix}_motor">
+    <hardwareInterface>hardware_interface/VelocityJointInterface</hardwareInterface>
+    <mechanicalReduction>1</mechanicalReduction>
+  </actuator>
+</transmission>
+</xacro:macro>
 <!-- define links -->
+<!-- dumy foot print -->
+<link name="base_foot_print">
+  <visual>
+    <origin xyz="0 0 0" rpy="0 0 0" />
+    <geometry>
+      <box size="0.001 0.001 0.001" />
+    </geometry>
+  </visual>
+</link>
+<gazebo reference="base_footprint">
+  <turnGravityOff>false</turnGravityOff>
+</gazebo>
+<joint name="base_footprint_joint" type="fixed">
+  <origin xyz="0 0 ${wheel_radius}" rpy="0 0 0" />
+  <parent link="base_foot_print"/>
+  <child link="base_link" />
+</joint>
 <!-- Base Link-->
 <link name="base_link">
@@ -36,59 +110,9 @@
 </gazebo>
 <!-- Left Wheel Link -->
-<link name="left_wheel_link">
-  <collision>
-    <geometry>
-      <cylinder length="${wheel_thickness}" radius="${wheel_radius}" />
-    </geometry>
-    <origin xyz="0 0 0" rpy="0 ${PI/2} 0" />
-  </collision>
-  <visual>
-    <geometry>
-      <cylinder length="${wheel_thickness}" radius="${wheel_radius}" />
-    </geometry>
-    <origin xyz="0 0 0" rpy="0 ${PI/2} 0" />
-    <material name="blue">
-      <color rgba="0 0 .8 1"/>
-    </material>
-  </visual>
-</link>
-<gazebo reference="left_wheel_link">
-  <material>Gazebo/Black</material>
-</gazebo>
-<joint name="left_wheel_joint" type="continuous">
-  <parent link="base_link" />
-  <child link="left_wheel_link" />
-  <origin xyz="${width/2} 0 ${wheel_radius}" rpy="0 0 0" />
-  <axis xyz="1 0 0" />
-</joint>
-<!-- Right wheel Link -->
-<link name="right_wheel_link">
-  <collision>
-    <geometry>
-      <cylinder length="${wheel_thickness}" radius="${wheel_radius}" />
-    </geometry>
-    <origin xyz="0 0 0" rpy="0 ${PI/2} 0" />
-  </collision>
-  <visual>
-    <geometry>
-      <cylinder length="${wheel_thickness}" radius="${wheel_radius}" />
-    </geometry>
-    <origin xyz="0 0 0" rpy="0 ${PI/2} 0" />
-    <material name="blue">
-      <color rgba="0 0 .8 1"/>
-    </material>
-  </visual>
-</link>
-<gazebo reference="right_wheel_link">
-  <material>Gazebo/Blue</material>
-</gazebo>
-<joint name="right_wheel_joint" type="continuous">
-  <parent link="base_link" />
-  <child link="right_wheel_link" />
-  <origin xyz="${-width/2} 0 ${wheel_radius}" rpy="0 0 0" />
-  <axis xyz="1 0 0" />
-</joint>
+<wheel_ prefix="left" reflect="-1" />
+<!-- Right Wheel Link -->
+<wheel_ prefix="right" reflect="1" />
 <!-- front caster link -->
-<link name="front_caster_link">
+<!--link name="front_caster_link">
   <visual>
     <geometry>
@@ -100,13 +124,13 @@
     </material>
   </visual>
-</link>
-<joint name="joint_front_caster" type="continuous">
+</link-->
+<!--joint name="joint_front_caster" type="continuous">
 <parent link="base_link" />
 <child link="front_caster_link" />
 <origin xyz="0 ${height/2} ${(wheel_radius - thickness/2)/2}" rpy="0 0 0" />
 <axis xyz="1 0 0" />
-</joint>
+</joint-->
 <!-- back caster link -->
-<link name="back_caster_link">
+<!--link name="back_caster_link">
   <visual>
     <geometry>
@@ -118,31 +142,11 @@
     </material>
   </visual>
-</link>
-<joint name="joint_back_caster" type="continuous">
+</link-->
+<!--joint name="joint_back_caster" type="continuous">
 <parent link="base_link" />
 <child link="back_caster_link" />
 <origin xyz="0 ${-height/2} ${(wheel_radius - thickness/2)/2}" rpy="0 0 0" />
 <axis xyz="1 0 0" />
-</joint>
-<transmission name="left_tran">
-  <type>transmission_interface/SimpleTransmission</type>
-  <joint name="left_whell_joint">
-    <hardwareInterface>hardware_interface/VelocityJointInterface</hardwareInterface>
-  </joint>
-  <actuator name="left_motor">
-    <hardwareInterface>hardware_interface/VelocityJointInterface</hardwareInterface>
-    <mechanicalReduction>1</mechanicalReduction>
-  </actuator>
-</transmission>
-<transmission name="right_tran">
-  <type>transmission_interface/SimpleTransmission</type>
-  <joint name="right_whell_joint">
-    <hardwareInterface>hardware_interface/VelocityJointInterface</hardwareInterface>
-  </joint>
-  <actuator name="right_motor">
-    <hardwareInterface>hardware_interface/VelocityJointInterface</hardwareInterface>
-    <mechanicalReduction>1</mechanicalReduction>
-  </actuator>
-</transmission>
+</joint-->
 <!-- ros_control plugin -->
 <!--
@@ -155,3 +159,28 @@
  </gazebo>
 -->
+ <!-- controller -->
+      <!--gazebo>
+        <plugin name="differential_drive_controller"
+                filename="libgazebo_ros_diff_drive.so">
+          <rosDebugLevel>Debug</rosDebugLevel>
+          <publishWheelTF>true</publishWheelTF>
+          <robotNamespace>/</robotNamespace>
+          <publishTf>1</publishTf>
+          <publishWheelJointState>true</publishWheelJointState>
+          <alwaysOn>true</alwaysOn>
+          <updateRate>100.0</updateRate>
+          <legacyMode>true</legacyMode>
+          <leftJoint>left_wheel_joint</leftJoint>
+          <rightJoint>right_wheel_joint</rightJoint>
+          <wheelSeparation>${width + wheel_thickness}</wheelSeparation>
+          <wheelDiameter>${2*wheel_radius}</wheelDiameter>
+          <broadcastTF>1</broadcastTF>
+          <wheelTorque>30</wheelTorque>
+          <wheelAcceleration>1.8</wheelAcceleration>
+          <commandTopic>cmd_vel</commandTopic>
+          <odometryFrame>odom</odometryFrame>
+          <odometryTopic>odom</odometryTopic>
+          <robotBaseFrame>base_footprint_joint</robotBaseFrame>
+        </plugin>
+      </gazebo-->
 </robot>

Commit message: 純粹利用 ros diff control plugin 控制車子

File: my_diffcar/urdf/diffcar.xacro (robot description, xacro)
@@ -10,4 +10,6 @@
 <xacro:property name="wheel_thickness" value="0.02" /> <!-- 1 cm -->
 <xacro:property name="wheel_radius" value="0.05" /> <!-- 5 cm -->
+<xacro:property name="caster_radius" value="${(wheel_radius - thickness/2)/2}" />
+<xacro:property name="caster_mass" value="0.1" /> <!-- kg -->
 <!-- define macros -->
 <xacro:macro name="sphere_inertial_matrix_" params="m r">
@@ -66,4 +68,33 @@
 </transmission>
 </xacro:macro>
+<xacro:macro name="caster_" params="prefix reflect">
+<link name="${prefix}_caster_link">
+  <visual>
+    <origin xyz="0 0 0" rpy="0 0 0"/>
+      <geometry>
+        <sphere radius="${caster_radius}" />
+      </geometry>
+      <material name="black">
+        <color rgba="0 0 0 1"/>
+      </material>
+  </visual>
+  <collision>
+    <origin xyz="0 0 0" rpy="0 0 0"/>
+      <geometry>
+        <sphere radius="${caster_radius}" />
+      </geometry>
+  </collision>
+    <sphere_inertial_matrix_  m="${caster_mass}" r="${caster_radius}" />
+  </link>
+  <joint name="${prefix}_caster_joint" type="continuous">
+  <origin xyz="0 ${reflect*(height/2 - caster_radius)} ${caster_radius}" rpy="0 0 0"/>
+    <parent link="base_link"/>
+    <child link="${prefix}_caster_link"/>
+    <axis xyz="1 0 0"/>
+  </joint>
+  <gazebo reference="${prefix}_caster_link">
+    <material>Gazebo/Black</material>
+  </gazebo>
+</xacro:macro>
 <!-- define links -->
 <!-- dumy foot print -->
@@ -114,39 +145,7 @@
 <wheel_ prefix="right" reflect="1" />
 <!-- front caster link -->
-<!--link name="front_caster_link">
-  <visual>
-    <geometry>
-      <sphere radius="${(wheel_radius - thickness/2)/2}" />
-    </geometry>
-    <origin xyz="0 0 0" rpy="0 0 0" />
-    <material name="black">
-      <color rgba="0 0 0 1"/>
-    </material>
-  </visual>
-</link-->
-<!--joint name="joint_front_caster" type="continuous">
-<parent link="base_link" />
-<child link="front_caster_link" />
-<origin xyz="0 ${height/2} ${(wheel_radius - thickness/2)/2}" rpy="0 0 0" />
-<axis xyz="1 0 0" />
-</joint-->
+<caster_ prefix="front" reflect="1" />
 <!-- back caster link -->
-<!--link name="back_caster_link">
-  <visual>
-    <geometry>
-      <sphere radius="${(wheel_radius - thickness/2)/2}" />
-    </geometry>
-    <origin xyz="0 0 0" rpy="0 0 0" />
-    <material name="black">
-      <color rgba="0 0 0 1"/>
-    </material>
-  </visual>
-</link-->
-<!--joint name="joint_back_caster" type="continuous">
-<parent link="base_link" />
-<child link="back_caster_link" />
-<origin xyz="0 ${-height/2} ${(wheel_radius - thickness/2)/2}" rpy="0 0 0" />
-<axis xyz="1 0 0" />
-</joint-->
+<caster_ prefix="back" reflect="-1" />
 <!-- ros_control plugin -->
 <!--
@@ -159,28 +158,29 @@
  </gazebo>
 -->
- <!-- controller -->
-      <!--gazebo>
-        <plugin name="differential_drive_controller"
-                filename="libgazebo_ros_diff_drive.so">
-          <rosDebugLevel>Debug</rosDebugLevel>
-          <publishWheelTF>true</publishWheelTF>
-          <robotNamespace>/</robotNamespace>
-          <publishTf>1</publishTf>
-          <publishWheelJointState>true</publishWheelJointState>
-          <alwaysOn>true</alwaysOn>
-          <updateRate>100.0</updateRate>
-          <legacyMode>true</legacyMode>
-          <leftJoint>left_wheel_joint</leftJoint>
-          <rightJoint>right_wheel_joint</rightJoint>
-          <wheelSeparation>${width + wheel_thickness}</wheelSeparation>
-          <wheelDiameter>${2*wheel_radius}</wheelDiameter>
-          <broadcastTF>1</broadcastTF>
-          <wheelTorque>30</wheelTorque>
-          <wheelAcceleration>1.8</wheelAcceleration>
-          <commandTopic>cmd_vel</commandTopic>
-          <odometryFrame>odom</odometryFrame>
-          <odometryTopic>odom</odometryTopic>
-          <robotBaseFrame>base_footprint_joint</robotBaseFrame>
-        </plugin>
-      </gazebo-->
+ <!-- gazebo controller plugin-->
+ <!-- ref:https://kiranpalla.com/autonomous-navigation-ros-differential-drive-robot-simulation/simple-navigation-with-differential-drive-plugin/-->
+<gazebo>
+<plugin name="differential_drive_controller"
+        filename="libgazebo_ros_diff_drive.so">
+  <rosDebugLevel>Debug</rosDebugLevel>
+  <publishWheelTF>true</publishWheelTF>
+  <robotNamespace>/</robotNamespace>
+  <publishTf>1</publishTf>
+  <publishWheelJointState>true</publishWheelJointState>
+  <alwaysOn>true</alwaysOn>
+  <updateRate>100.0</updateRate>
+  <legacyMode>true</legacyMode>
+  <leftJoint>left_wheel_joint</leftJoint>
+  <rightJoint>right_wheel_joint</rightJoint>
+  <wheelSeparation>${width + wheel_thickness}</wheelSeparation>
+  <wheelDiameter>${2*wheel_radius}</wheelDiameter>
+  <broadcastTF>1</broadcastTF>
+  <wheelTorque>30</wheelTorque>
+  <wheelAcceleration>1.8</wheelAcceleration>
+  <commandTopic>cmd_vel</commandTopic>
+  <odometryFrame>odom</odometryFrame>
+  <odometryTopic>odom</odometryTopic>
+  <robotBaseFrame>base_footprint_joint</robotBaseFrame>
+</plugin>
+</gazebo>
 </robot>

Commit message: 1. 不可 remap /joint_states，這樣 tf 才能整卻關聯; 2. 修正 joint 位置，應該以 parent 為基準點

File: my_diffcar/urdf/diffcar.xacro (robot description, xacro)
@@ -13,4 +13,12 @@
 <xacro:property name="caster_mass" value="0.1" /> <!-- kg -->
 <!-- define macros -->
+<xacro:macro name="box_inertia_matrix_" params="m w h d">
+  <inertial>
+    <mass value="${m}"/>
+    <inertia ixx="${m / 12.0 * (d*d + h*h)}" ixy="0.0" ixz="0.0"
+             iyy="${m / 12.0 * (w*w + h*h)}" iyz="0.0"
+             izz="${m / 12.0 * (w*w + d*d)}"/>
+  </inertial>
+</xacro:macro>
 <xacro:macro name="sphere_inertial_matrix_" params="m r">
   <inertial>
@@ -54,10 +62,10 @@
   <parent link="base_link" />
   <child link="${prefix}_wheel_link" />
-  <origin xyz="${(width/2 + wheel_thickness/2)*reflect} 0 ${wheel_radius}" rpy="0 0 0" />
+  <origin xyz="${(width/2 + wheel_thickness/2)*reflect} 0 0" rpy="0 0 0" />
   <axis xyz="1 0 0" />
 </joint>
 <transmission name="${prefix}_tran">
   <type>transmission_interface/SimpleTransmission</type>
-  <joint name="${prefix}_whell_joint">
+  <joint name="${prefix}_wheel_joint">
     <hardwareInterface>hardware_interface/VelocityJointInterface</hardwareInterface>
   </joint>
@@ -88,7 +96,7 @@
   </link>
   <joint name="${prefix}_caster_joint" type="continuous">
-  <origin xyz="0 ${reflect*(height/2 - caster_radius)} ${caster_radius}" rpy="0 0 0"/>
     <parent link="base_link"/>
     <child link="${prefix}_caster_link"/>
+    <origin xyz="0 ${reflect*(height/2 - caster_radius)} ${-(caster_radius + thickness/2)}" rpy="0 0 0"/>
     <axis xyz="1 0 0"/>
   </joint>
@@ -98,6 +106,6 @@
 </xacro:macro>
 <!-- define links -->
-<!-- dumy foot print -->
-<link name="base_foot_print">
+<!-- base foot print -->
+<link name="base_footprint">
   <visual>
     <origin xyz="0 0 0" rpy="0 0 0" />
@@ -106,13 +114,9 @@
     </geometry>
   </visual>
+  <box_inertia_matrix_ m="${mass*2}" w="0.001" h="0.001" d="0.001" />
 </link>
 <gazebo reference="base_footprint">
   <turnGravityOff>false</turnGravityOff>
 </gazebo>
-<joint name="base_footprint_joint" type="fixed">
-  <origin xyz="0 0 ${wheel_radius}" rpy="0 0 0" />
-  <parent link="base_foot_print"/>
-  <child link="base_link" />
-</joint>
 <!-- Base Link-->
 <link name="base_link">
@@ -121,5 +125,4 @@
       <box size="${width} ${height} ${thickness}" />
     </geometry>
-    <origin xyz="0 0 ${wheel_radius}" rpy="0 0 0" />
   </collision>
   <visual>
@@ -127,14 +130,12 @@
       <box size="${width} ${height} ${thickness}" />
     </geometry>
-    <origin xyz="0 0 ${wheel_radius}" rpy="0 0 0" />
   </visual>
-  <inertial>
-    <mass value="${mass}" />
-    <inertia
-	  ixx="${mass / 12.0 * (width*height + thickness*thickness)}" ixy="0.0" ixz="0.0"
-	  iyy="${mass / 12.0 * (thickness*thickness + width*height)}" iyz="0.0"
-	  izz="${mass / 12.0 * (width*height + width*height)}"/>
-  </inertial>
+  <box_inertia_matrix_ m="${mass}" w="${width}" h="${height}" d="${thickness}" />
 </link>
+<joint name="base_link_joint" type="fixed">
+  <origin xyz="0 0 ${wheel_radius}" rpy="0 0 0" />
+  <parent link="base_footprint"/>
+  <child link="base_link" />
+</joint>
 <gazebo reference="base_link">
   <material>Gazebo/Orange</material>
@@ -148,16 +149,6 @@
 <!-- back caster link -->
 <caster_ prefix="back" reflect="-1" />
-<!-- ros_control plugin -->
-<!--
- <gazebo>
-   <plugin name="gazebo_ros_control" filename="libgazebo_ros_control.so">
-     <robotNamespace>/rotor</robotNamespace>
-     <robotSimType>gazebo_ros_control/DefaultRobotHWSim</robotSimType>
-     <legacyModeNS>true</legacyModeNS>
-   </plugin>
- </gazebo>
--->
- <!-- gazebo controller plugin-->
- <!-- ref:https://kiranpalla.com/autonomous-navigation-ros-differential-drive-robot-simulation/simple-navigation-with-differential-drive-plugin/-->
+<!-- gazebo controller plugin-->
+<!-- ref:https://kiranpalla.com/autonomous-navigation-ros-differential-drive-robot-simulation/simple-navigation-with-differential-drive-plugin/-->
 <gazebo>
 <plugin name="differential_drive_controller"
@@ -181,5 +172,5 @@
   <odometryFrame>odom</odometryFrame>
   <odometryTopic>odom</odometryTopic>
-  <robotBaseFrame>base_footprint_joint</robotBaseFrame>
+  <robotBaseFrame>base_footprint</robotBaseFrame>
 </plugin>
 </gazebo>

Commit message: 加入 ros 控制器，測試成功

File: my_diffcar/urdf/diffcar.xacro (robot description, xacro)
@@ -1,4 +1,4 @@
 <?xml version="1.0"?>
-<robot name="rotor" xmlns:xacro="http://www.ros.org/wiki/xacro">
+<robot name="diffcar" xmlns:xacro="http://www.ros.org/wiki/xacro">
 <!-- define constants -->
 <xacro:property name="PI" value="3.1415926" />

File: my_rosdiffcar/urdf/rosdiffcar.xacro (robot description, xacro)
@@ -1,12 +1,12 @@
 <?xml version="1.0"?>
-<robot name="rotor" xmlns:xacro="http://www.ros.org/wiki/xacro">
+<robot name="rosdiffcar" xmlns:xacro="http://www.ros.org/wiki/xacro">
 <!-- define constants -->
 <xacro:property name="PI" value="3.1415926" />
 <xacro:property name="mass" value="1" /> <!-- kg -->
 <xacro:property name="wheel_mass" value="0.3" /> <!-- kg -->
-<xacro:property name="width" value="0.2" /> <!-- 0.1m -->
-<xacro:property name="height" value="0.4" /> <!-- 0.2m -->
+<xacro:property name="width" value="0.2" /> <!-- 0.2m -->
+<xacro:property name="height" value="0.4" /> <!-- 0.4m -->
 <xacro:property name="thickness" value="0.02" /> <!-- 2 cm -->
-<xacro:property name="wheel_thickness" value="0.02" /> <!-- 1 cm -->
+<xacro:property name="wheel_thickness" value="0.02" /> <!-- 2 cm -->
 <xacro:property name="wheel_radius" value="0.05" /> <!-- 5 cm -->
 <xacro:property name="caster_radius" value="${(wheel_radius - thickness/2)/2}" />
@@ -153,5 +153,4 @@
 <gazebo>
   <plugin name="gazebo_ros_control" filename="libgazebo_ros_control.so">
-    <robotNamespace>/rosdiffcar</robotNamespace>
     <robotSimType>gazebo_ros_control/DefaultRobotHWSim</robotSimType>
     <legacyModeNS>true</legacyModeNS>
