Commit message: 新增 showurdf.sh

File: my_slider/urdf/slider.xacro (robot description, xacro)
@@ -7,4 +7,8 @@
 <xacro:property name="height1" value="2" /> <!-- 2m -->
 <xacro:property name="height2" value="1" /> <!-- 1m -->
+<!-- define colors -->
+<material name="blue">
+  <color rgba="0 0 0.8 1" />
+</material>
 <!-- define links -->
 <link name="world" />
@@ -47,4 +51,5 @@
       <box size="${width} ${width} ${height2}" />
     </geometry>
+    <material name="blue" />
     <origin xyz="0 0 ${height2/2}" rpy="0 0 0" />
   </visual>

Commit message: 完成導入控制器

File: my_slider/urdf/slider.xacro (robot description, xacro)
@@ -7,8 +7,4 @@
 <xacro:property name="height1" value="2" /> <!-- 2m -->
 <xacro:property name="height2" value="1" /> <!-- 1m -->
-<!-- define colors -->
-<material name="blue">
-  <color rgba="0 0 0.8 1" />
-</material>
 <!-- define links -->
 <link name="world" />
@@ -35,4 +31,7 @@
   </inertial>
 </link>
+<gazebo reference="link1">
+  <material>Gazebo/Orange</material>
+</gazebo>
 <joint name="ground_joint" type="fixed">  <!-- fix to the ground -->
   <parent link="world" />
@@ -51,5 +50,4 @@
       <box size="${width} ${width} ${height2}" />
     </geometry>
-    <material name="blue" />
     <origin xyz="0 0 ${height2/2}" rpy="0 0 0" />
   </visual>
@@ -62,5 +60,8 @@
   </inertial>
 </link>
-<joint name="link1_2_joint" type="prismatic">
+<gazebo reference="link2">
+  <material>Gazebo/Black</material>
+</gazebo>
+<joint name="joint1" type="prismatic">
   <parent link="link1" />
   <child link="link2" />
@@ -79,3 +80,11 @@
   </actuator>
 </transmission>
+<!-- ros_control plugin -->
+ <gazebo>
+   <plugin name="gazebo_ros_control" filename="libgazebo_ros_control.so">
+     <robotNamespace>/slider</robotNamespace>
+     <robotSimType>gazebo_ros_control/DefaultRobotHWSim</robotSimType>
+     <legacyModeNS>true</legacyModeNS>  <!-- KC_DBG : to avoid gazebo version warring-->
+   </plugin>
+ </gazebo>
 </robot>

Commit message: 將 link1 改為 base_link，避免 rviz 啟用錯誤

File: my_slider/urdf/slider.xacro (robot description, xacro)
@@ -10,5 +10,5 @@
 <link name="world" />
 <!-- Base Link-->
-<link name="link1">
+<link name="base_link">
   <collision>
     <geometry>
@@ -31,10 +31,10 @@
   </inertial>
 </link>
-<gazebo reference="link1">
+<gazebo reference="base_link">
   <material>Gazebo/Orange</material>
 </gazebo>
 <joint name="ground_joint" type="fixed">  <!-- fix to the ground -->
   <parent link="world" />
-  <child link="link1" />
+  <child link="base_link" />
 </joint>
 <!-- Link 2 -->
@@ -64,5 +64,5 @@
 </gazebo>
 <joint name="joint1" type="prismatic">
-  <parent link="link1" />
+  <parent link="base_link" />
   <child link="link2" />
   <limit effort="100" velocity="0.1" lower="-1.0" upper="1.0" />

Commit message: slider 改用 velocity/position contoller，可以上下速度穩定

File: my_slider/urdf/slider.xacro (robot description, xacro)
@@ -66,5 +66,5 @@
   <parent link="base_link" />
   <child link="link2" />
-  <limit effort="100" velocity="0.1" lower="-1.0" upper="1.0" />
+  <limit effort="100" velocity="0.2" lower="-1.0" upper="1.0" />
   <origin xyz="0 ${width} ${height1/2}" rpy="0 0 0" />
   <axis xyz="0 0 1" />
@@ -73,8 +73,8 @@
   <type>transmission_interface/SimpleTransmission</type>
   <joint name="joint1">
-    <hardwareInterface>hardware_interface/EffortJointInterface</hardwareInterface>
+    <hardwareInterface>hardware_interface/VelocityJointInterface</hardwareInterface>
   </joint>
   <actuator name="motor1">
-    <hardwareInterface>hardware_interface/EffortJointInterface</hardwareInterface>
+    <hardwareInterface>hardware_interface/VelocityJointInterface</hardwareInterface>
     <mechanicalReduction>1</mechanicalReduction>
   </actuator>
