Commit message: 三輪車加入轉盤位置控制器、舵輪速度控制器

File: my_tricycle/urdf/tricycle.xacro (robot description, xacro)
@@ -68,14 +68,4 @@
   <axis xyz="1 0 0" />
 </joint>
-<transmission name="${prefix}_tran">
-  <type>transmission_interface/SimpleTransmission</type>
-  <joint name="${prefix}_wheel_joint">
-    <hardwareInterface>hardware_interface/VelocityJointInterface</hardwareInterface>
-  </joint>
-  <actuator name="${prefix}_motor">
-    <hardwareInterface>hardware_interface/VelocityJointInterface</hardwareInterface>
-    <mechanicalReduction>1</mechanicalReduction>
-  </actuator>
-</transmission>
 </xacro:macro>
 <!-- define links -->
@@ -167,4 +157,14 @@
   <axis xyz="0 0 1" />
 </joint>
+<transmission name="disk_tran">
+  <type>transmission_interface/SimpleTransmission</type>
+  <joint name="disk_link_joint">
+    <hardwareInterface>hardware_interface/PositionJointInterface</hardwareInterface>
+  </joint>
+  <actuator name="disk_motor">
+    <hardwareInterface>hardware_interface/PositionJointInterface</hardwareInterface>
+    <mechanicalReduction>1</mechanicalReduction>
+  </actuator>
+</transmission>
 <!-- steer_wheel -->
 <link name="steer_wheel_link">
@@ -195,4 +195,14 @@
   <axis xyz="1 0 0" />
 </joint>
+<transmission name="steer_tran">
+  <type>transmission_interface/SimpleTransmission</type>
+  <joint name="steer_wheel_joint">
+    <hardwareInterface>hardware_interface/VelocityJointInterface</hardwareInterface>
+  </joint>
+  <actuator name="steer_motor">
+    <hardwareInterface>hardware_interface/VelocityJointInterface</hardwareInterface>
+    <mechanicalReduction>1</mechanicalReduction>
+  </actuator>
+</transmission>
 <!-- gazebo controller plugin: ref: http://gazebosim.org/tutorials/?tut=ros_control-->
 <!-- ref: http://www.theconstructsim.com/ros-qa-126-how-to-configure-the-differential-drive-ros-controller/-->

Commit message: 新增三輪車舵輪耳朵

File: my_tricycle/urdf/tricycle.xacro (robot description, xacro)
@@ -15,4 +15,7 @@
 <xacro:property name="disk_radius" value="${(stick_width - thickness*2)/2}" />
 <xacro:property name="disk_thickness" value="${thickness/2}" />
+<xacro:property name="ear_width" value="${disk_radius}" />
+<xacro:property name="ear_height" value="${disk_radius*2}" />
+<xacro:property name="ear_thickness" value="${thickness/2}" />
 <!-- define macros -->
 <xacro:macro name="box_inertia_matrix_" params="m w h d">
@@ -66,4 +69,27 @@
   <child link="${prefix}_wheel_link" />
   <origin xyz="${(width/2 + wheel_thickness/2)*reflect} 0 0" rpy="0 0 0" />
+  <axis xyz="1 0 0" />
+</joint>
+</xacro:macro>
+<xacro:macro name="ear_" params="prefix reflect">
+<link name="${prefix}_ear_link">
+  <visual>
+    <geometry>
+      <box size="${ear_width} ${ear_height} ${ear_thickness}" />
+    </geometry>
+    <origin xyz="0 0 0" rpy="${PI/2} 0 ${PI/2}" />
+  </visual>
+  <collision>
+    <geometry>
+      <box size="${ear_width} ${ear_height} ${ear_thickness}" />
+    </geometry>
+    <origin xyz="0 0 0" rpy="${PI/2} 0 ${PI/2}" />
+  </collision>
+  <box_inertia_matrix_  m="${mass*0.1}" w="${ear_width}" h="${ear_height}" d="${ear_thickness}"/>
+</link>
+<joint name="${prefix}_ear_joint" type="fixed">
+  <parent link="disk_link" />
+  <child link="${prefix}_ear_link" />
+  <origin xyz="${(disk_radius + ear_thickness/2)*reflect} 0 ${-ear_height/2 + disk_thickness/2}" rpy="0 0 0" />
   <axis xyz="1 0 0" />
 </joint>
@@ -132,4 +158,8 @@
   <child link="stick_link" />
 </joint>
+<!--  left ear -->
+<ear_ prefix="left" reflect="-1" />
+<!--  right ear -->
+<ear_ prefix="right" reflect="1" />
 <!-- disk -->
 <link name="disk_link">
