Commit message: 加重;留間距避免舵輪摩擦、震盪;調整 pid 讓輪向穩定

File: my_rostricycle/urdf/rostricycle.xacro (robot description, xacro)
@@ -3,11 +3,11 @@
 <!-- define constants -->
 <xacro:property name="PI" value="3.1415926" />
-<xacro:property name="mass" value="1" />
-<xacro:property name="wheel_mass" value="0.3" />
-<xacro:property name="width" value="0.2" />
-<xacro:property name="height" value="0.4" />
-<xacro:property name="thickness" value="0.02" />
-<xacro:property name="wheel_thickness" value="0.02" />
-<xacro:property name="wheel_radius" value="0.05" />
+<xacro:property name="mass" value="5" />
+<xacro:property name="wheel_mass" value="1.5" />
+<xacro:property name="width" value="1" />
+<xacro:property name="height" value="2" />
+<xacro:property name="thickness" value="0.1" />
+<xacro:property name="wheel_thickness" value="0.1" />
+<xacro:property name="wheel_radius" value="0.25" />
 <xacro:property name="stick_width" value="${(wheel_thickness)*4}" />
 <xacro:property name="stick_height" value="${(wheel_radius)*4}" />
@@ -156,4 +156,7 @@
 <!--  left ear -->
 <ear_ prefix="left" reflect="-1" />
+<gazebo reference="left_ear_link">
+  <material>Gazebo/Red</material>
+</gazebo>
 <!--  right ear -->
 <ear_ prefix="right" reflect="1" />
@@ -218,5 +221,5 @@
   <parent link="disk_link" />
   <child link="steer_wheel_link" />
-  <origin xyz="0 0 ${-wheel_radius/2 - disk_thickness/2}" rpy="0 0 0" />
+  <origin xyz="0 0 ${-wheel_radius/2 - disk_thickness/2 - disk_thickness/2}" rpy="0 0 0" />
   <axis xyz="1 0 0" />
 </joint>

Commit message: 新增舵輪標記點、排除 gazebo 啟動警告

File: my_rostricycle/urdf/rostricycle.xacro (robot description, xacro)
@@ -234,4 +234,28 @@
   </actuator>
 </transmission>
+<!-- steer_wheel_mark -->
+<link name="steer_wheel_mark_link">
+  <visual>
+    <geometry>
+      <cylinder length="0.01" radius="0.01" />
+    </geometry>
+    <origin xyz="0 0 0" rpy="0 ${PI/2} 0" />
+    <material name="white">
+      <color rgba=".8 .8 .8 1"/>
+    </material>
+  </visual>
+  <collision>
+    <geometry>
+      <cylinder length="0.01" radius="0.01" />
+    </geometry>
+    <origin xyz="0 0 0" rpy="0 ${PI/2} 0" />
+  </collision>
+</link>
+<joint name="steer_wheel_mark_joint" type="fixed">
+  <parent link="steer_wheel_link" />
+  <child link="steer_wheel_mark_link" />
+  <origin xyz="${wheel_thickness/2+0.005} 0  ${wheel_radius/2-0.01}" rpy="0 0 0" />
+  <axis xyz="1 0 0" />
+</joint>
 <!-- gazebo controller plugin: ref: http://gazebosim.org/tutorials/?tut=ros_control-->
 <!-- ref: http://www.theconstructsim.com/ros-qa-126-how-to-configure-the-differential-drive-ros-controller/-->

Commit message: 調整舵輪關節名稱，並增加硬體驅動器

File: my_rostricycle/urdf/rostricycle.xacro (robot description, xacro)
@@ -13,8 +13,8 @@
 <xacro:property name="stick_height" value="${(wheel_radius)*4}" />
 <xacro:property name="stick_thickness" value="${thickness}" />
-<xacro:property name="disk_radius" value="${(stick_width - thickness*2)/2}" />
-<xacro:property name="disk_thickness" value="${thickness/2}" />
-<xacro:property name="ear_width" value="${disk_radius}" />
-<xacro:property name="ear_height" value="${disk_radius*2}" />
+<xacro:property name="steer_radius" value="${(stick_width - thickness*2)/2}" />
+<xacro:property name="steer_thickness" value="${thickness/2}" />
+<xacro:property name="ear_width" value="${steer_radius}" />
+<xacro:property name="ear_height" value="${steer_radius*2}" />
 <xacro:property name="ear_thickness" value="${thickness/2}" />
 <!-- define macros -->
@@ -89,7 +89,7 @@
 </link>
 <joint name="${prefix}_ear_joint" type="fixed">
-  <parent link="disk_link" />
+  <parent link="front_steering_link" />
   <child link="${prefix}_ear_link" />
-  <origin xyz="${(disk_radius + ear_thickness/2)*reflect} 0 ${-ear_height/2 + disk_thickness/2}" rpy="0 0 0" />
+  <origin xyz="${(steer_radius + ear_thickness/2)*reflect} 0 ${-ear_height/2 + steer_thickness/2}" rpy="0 0 0" />
   <axis xyz="1 0 0" />
 </joint>
@@ -161,9 +161,9 @@
 <!--  right ear -->
 <ear_ prefix="right" reflect="1" />
-<!-- disk -->
-<link name="disk_link">
-  <visual>
-    <geometry>
-      <cylinder length="${disk_thickness}" radius="${disk_radius}" />
+<!-- front steer -->
+<link name="front_steering_link">
+  <visual>
+    <geometry>
+      <cylinder length="${steer_thickness}" radius="${steer_radius}" />
     </geometry>
     <origin xyz="0 0 0" rpy="0 0 0" />
@@ -174,28 +174,28 @@
   <collision>
     <geometry>
-      <cylinder length="${disk_thickness}" radius="${disk_radius}" />
+      <cylinder length="${steer_thickness}" radius="${steer_radius}" />
     </geometry>
     <origin xyz="0 0 0" rpy="0 0 0" />
   </collision>
-  <cylinder_inertial_matrix_  m="${wheel_mass/2}" r="${disk_radius}" h="${disk_thickness}" />
-</link>
-<joint name="disk_link_joint" type="continuous">
+  <cylinder_inertial_matrix_  m="${wheel_mass/2}" r="${steer_radius}" h="${steer_thickness}" />
+</link>
+<joint name="front_steering_joint" type="continuous">
   <parent link="stick_link" />
-  <child link="disk_link" />
-  <origin xyz="0 ${-stick_height/2 + disk_radius} ${-stick_thickness/2 - disk_thickness/2}" rpy="0 0 0" />
+  <child link="front_steering_link" />
+  <origin xyz="0 ${-stick_height/2 + steer_radius} ${-stick_thickness/2 - steer_thickness/2}" rpy="0 0 0" />
   <axis xyz="0 0 1" />
 </joint>
-<transmission name="disk_tran">
+<transmission name="front_steering_tran">
   <type>transmission_interface/SimpleTransmission</type>
-  <joint name="disk_link_joint">
+  <joint name="front_steering_joint">
     <hardwareInterface>hardware_interface/PositionJointInterface</hardwareInterface>
   </joint>
-  <actuator name="disk_motor">
+  <actuator name="front_steering_motor">
     <hardwareInterface>hardware_interface/PositionJointInterface</hardwareInterface>
     <mechanicalReduction>1</mechanicalReduction>
   </actuator>
 </transmission>
-<!-- steer_wheel -->
-<link name="steer_wheel_link">
+<!-- front wheel -->
+<link name="front_wheel_link">
   <visual>
     <geometry>
@@ -215,25 +215,25 @@
   <cylinder_inertial_matrix_  m="${wheel_mass/4}" r="${wheel_radius/2}" h="${wheel_thickness}" />
 </link>
-<gazebo reference="steer_wheel_link">
+<gazebo reference="front_wheel_link">
   <material>Gazebo/Yellow</material>
 </gazebo>
-<joint name="steer_wheel_joint" type="continuous">
-  <parent link="disk_link" />
-  <child link="steer_wheel_link" />
-  <origin xyz="0 0 ${-wheel_radius/2 - disk_thickness/2 - disk_thickness/2}" rpy="0 0 0" />
-  <axis xyz="1 0 0" />
-</joint>
-<transmission name="steer_tran">
+<joint name="front_wheel_joint" type="continuous">
+  <parent link="front_steering_link" />
+  <child link="front_wheel_link" />
+  <origin xyz="0 0 ${-wheel_radius/2 - steer_thickness/2 - steer_thickness/2}" rpy="0 0 0" />
+  <axis xyz="1 0 0" />
+</joint>
+<transmission name="front_wheel_tran">
   <type>transmission_interface/SimpleTransmission</type>
-  <joint name="steer_wheel_joint">
+  <joint name="front_wheel_joint">
     <hardwareInterface>hardware_interface/VelocityJointInterface</hardwareInterface>
   </joint>
-  <actuator name="steer_motor">
+  <actuator name="front_wheel_motor">
     <hardwareInterface>hardware_interface/VelocityJointInterface</hardwareInterface>
     <mechanicalReduction>1</mechanicalReduction>
   </actuator>
 </transmission>
-<!-- steer_wheel_mark -->
-<link name="steer_wheel_mark_link">
+<!-- front_wheel_mark -->
+<link name="front_wheel_mark_link">
   <visual>
     <geometry>
@@ -252,7 +252,7 @@
   </collision>
 </link>
-<joint name="steer_wheel_mark_joint" type="fixed">
-  <parent link="steer_wheel_link" />
-  <child link="steer_wheel_mark_link" />
+<joint name="front_wheel_mark_joint" type="fixed">
+  <parent link="front_wheel_link" />
+  <child link="front_wheel_mark_link" />
   <origin xyz="${wheel_thickness/2+0.005} 0  ${wheel_radius/2-0.01}" rpy="0 0 0" />
   <axis xyz="1 0 0" />

Commit message: 多個關節 vel handle，要註冊在同一個 joint_vel_interface_，才不會後令壓前令，找不到 resource

File: my_rostricycle/urdf/rostricycle.xacro (robot description, xacro)
@@ -258,4 +258,42 @@
   <axis xyz="1 0 0" />
 </joint>
+<!-- fork -->
+<link name="fork_link">
+  <visual>
+    <geometry>
+      <box size="${width/4} ${height/3} ${thickness}" />
+    </geometry>
+    <origin xyz="0 0 0" rpy="0 0 0" />
+    <material name="white">
+      <color rgba="0.8 0.8 0.8 1"/>
+    </material>
+  </visual>
+  <collision>
+    <geometry>
+      <box size="${width/4} ${height/3} ${thickness}" />
+    </geometry>
+    <origin xyz="0 0 0" rpy="0 0 0" />
+  </collision>
+  <box_inertia_matrix_  m="${mass*0.1}" w="${width/4}" h="${height/3}" d="${thickness}"/>
+</link>
+<joint name="fork_joint" type="prismatic">
+  <parent link="stick_link" />
+  <child link="fork_link" />
+  <limit effort="100.0" velocity="0.1" lower="0.0" upper="2.0"/>
+  <origin xyz=" 0 0 ${thickness}" rpy="0 0 0" />
+  <axis xyz="0 0 1" />
+</joint>
+<transmission name="fork_joint_trans">
+    <type>transmission_interface/SimpleTransmission</type>
+    <joint name="fork_joint">
+      <!--hardwareInterface>hardware_interface/EffortJointInterface</hardwareInterface-->
+      <hardwareInterface>hardware_interface/VelocityJointInterface</hardwareInterface>
+    </joint>
+    <actuator name="fork_actuator">
+      <!--hardwareInterface>hardware_interface/EffortJointInterface</hardwareInterface-->
+      <hardwareInterface>hardware_interface/VelocityJointInterface</hardwareInterface>
+      <mechanicalReduction>1</mechanicalReduction>
+    </actuator>
+</transmission>
 <!-- gazebo controller plugin: ref: http://gazebosim.org/tutorials/?tut=ros_control-->
 <!-- ref: http://www.theconstructsim.com/ros-qa-126-how-to-configure-the-differential-drive-ros-controller/-->

File: my_slider/urdf/slider.xacro (robot description, xacro)
@@ -63,5 +63,5 @@
   <material>Gazebo/Black</material>
 </gazebo>
-<joint name="joint1" type="prismatic">
+<joint name="fork_joint" type="prismatic">
   <parent link="base_link" />
   <child link="link2" />
@@ -72,5 +72,5 @@
 <transmission name="tran1">
   <type>transmission_interface/SimpleTransmission</type>
-  <joint name="joint1">
+  <joint name="fork_joint">
     <hardwareInterface>hardware_interface/VelocityJointInterface</hardwareInterface>
   </joint>
